File: boards/xbp/XBP.brd (EAGLE design)
At the start: 64.8 x 31.1 mm, 17 parts, among them IC1 MCP1701AT, U1 INA225

Commit message: version 2.0
Parts:
- removed JP3: GND, pinhead:1X01
- removed U$3, U$4: SILK_3V3_TAG, Public_BP_Library:SILK_3V3_TAG
- added JP5: Gain, pinhead:2X03
- added LED1: Power, led:CHIPLED_0603
- added LED2: Activity, led:CHIPLED_0603
- added Q1: BSS84, transistor-small-signal:SOT23
- added Q2, Q3, Q4, Q5, Q6, Q7, Q8: BSS123, transistor-small-signal:SOT23
- added R10, R11, R12, R7, R8, R9: 10k, resistor:R0603
- added R13: 22, resistor:R0603
- added R5: 1K, resistor:R0603
- added R6: 470, resistor:R0603
- added SJ2: SDA, jumper:SJ
- added SJ3: RST, jumper:SJ
- added SJ4: VCCH, jumper:SJ
- added SJ5: VCCP, jumper:SJ
- added U3, U4: SILK_3V3_TAG, Public_BP_Library:SILK_3V3_TAG
- added X1: SMA-142-0711-871/876, con-coax:J502-ND-142-0711-871/876
- A1: value (none) -> XBHCon
- A2: value (none) -> XBDCon
- JP1: value Vs 5V from XBH -> Power; device pinhead:1X02/90 -> pinhead:1X06/90
- JP2: value Vcc for XBD -> XBD; device pinhead:1X02/90 -> pinhead:2X04/90
- R1: value 10 -> 1R
- SJ1: value no IC1 -> SCL
- moved JP2 32.7 mm to (39.4, 30.5), turned to 0 degrees
- moved JP1 11.7 mm to (29.2, 0.64)
- moved IC1 8.60 mm to (21.0, 9.84)
- moved C2 6.93 mm to (20.6, 14.0)
- moved C3 6.79 mm to (20.6, 16.5)
- moved SJ1 5.91 mm to (21.6, 14.6), flipped to the bottom, turned to 270 degrees
- moved C1 4.87 mm to (25.1, 15.4), turned to 90 degrees
- moved U1 4.52 mm to (26.0, 20.6)
- moved R2 4.26 mm to (20.1, 20.7)
- moved R1 4.12 mm to (22.5, 20.6)
- moved R3 1.59 mm to (18.4, 5.08), flipped to the bottom, turned to 180 degrees
- moved R4 1.59 mm to (18.4, 2.54), flipped to the bottom, turned to 180 degrees
- moved A2 1.59 mm to (11.7, 16.5)
- moved A1 1.59 mm to (4.13, 16.5)
Connections:
- net TC1 renamed TF1
- net TC2 renamed TF2
- net TC3 renamed TF3
- removed net N$6: C2.1, C3.1, IC1.3, R1.1, R2.1, SJ1.2, U1.1
- removed net TC0: A1.36, A2.19
- new net N$10: Q1.1, Q2.3, R7.1
- new net N$12: Q7.3, Q8.1, R11.1
- new net N$3: LED1.A, R5.1
- new net N$7: Q3.3, Q4.3
- new net N$9: Q5.3, Q6.3
- new net RSTD: JP2.8, Q8.3, R10.1, SJ3.1
- new net SCLD: JP2.6, Q3.2, R8.1, SJ1.1
- new net SDAD: JP2.3, Q5.2, R9.1, SJ2.1
- new net TF0: A1.36, Q1.3, R6.2
- new net TF0D: A2.19, JP2.5, R13.2
- new net VCC: JP1.4, Q1.2, Q4.1, Q6.1, R11.2, R3.2, R4.2, R7.2, SJ4.1
- new net VCCD: A2.1, JP2.1, Q3.1, Q5.1, R1.2, R10.2, R2.2, R8.2, R9.2, U1.8
- new net VCCXBD: C2.1, C3.1, IC1.3, JP1.6, R1.1, R2.1, U1.1
- new net VCCXBP: C1.2, IC1.2@1, JP1.2, JP5.1, JP5.2, R5.2, SJ5.1, U1.3
- net GND: now also JP1.1, JP1.3, JP1.5, JP2.2, JP2.7, JP5.5, JP5.6, LED1.C, LED2.C, Q2.2, Q7.2, Q8.2, R12.1, X1.G@1, X1.G@2, X1.G@3, X1.G@4; no longer JP3.1
- net GS0: now also JP5.3
- net GS1: now also JP5.4
- net N$1: now also SJ4.2; no longer R3.2, R4.2
- net N$2: now also A1.21, SJ5.2; no longer A2.1, R1.2, R2.2, U1.8
- net N$4: now also Q2.1, R12.2, R13.1; no longer IC1.2@1, JP2.1, JP2.2, SJ1.1
- net N$5: now also LED2.A, R6.1; no longer C1.2, JP1.1, JP1.2, U1.3
- net PWR0: now also X1.1
- net RST0: now also Q7.1, SJ3.2
- net SCL: now also Q4.2, SJ1.2
- net SDA: now also Q6.2, SJ2.2
Routing:
- net VCCD: track 0.00 -> 63.8 mm, vias 0 -> 5
- net VCCXBP: track 0.00 -> 61.0 mm
- net VCC: track 0.00 -> 57.2 mm
- net SCLD: track 0.00 -> 33.0 mm, vias 0 -> 1
- net TF0D: track 0.00 -> 32.8 mm
- net VCCXBD: track 0.00 -> 31.5 mm
- net N$6: track 25.7 -> 0.00 mm
- net SDA: track 15.0 -> 38.6 mm, vias 0 -> 2
- net RST0: track 23.5 -> 46.9 mm, vias 0 -> 1
- net N$5: track 24.7 -> 2.21 mm
- net SDAD: track 0.00 -> 22.3 mm
- net RSTD: track 0.00 -> 21.2 mm
- net TF2: track 51.4 -> 70.7 mm
- net N$2: track 26.0 -> 42.8 mm
- net GND: track 26.4 -> 9.55 mm, vias 3 -> 8
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Other:
- board size 64.8 x 31.1 mm -> 61.3 x 31.1 mm
- board text added: "+"
- board text added: "0"
- board text added: "0b"
- board text added: "1"
- board text added: "10"
- board text added: "100"
- board text added: "11"
- board text added: "1a"
- board text added: "1b"
- board text added: "2"
- board text added: "20"
- board text added: "200"
- board text added: "21"
- board text added: "25"
- board text added: "2a"
- board text added: "2b"
- board text added: "3"
- board text added: "30"
- board text added: "31"
- board text added: "3a"
- board text added: "3b"
- board text added: "40"
- board text added: "50"
- board text added: "5V"
- board text added: "Activity"
- board text added: "C1"
- board text added: "C2"
- board text added: "C3"
- board text added: "GND"
- board text added: "GS0a"
- board text added: "GS1a"
- board text added: "GS2a"
- board text added: "GS3a"
- board text added: "GS3b"
- board text added: "Gain"
- board text added: "IC1"
- board text added: "J1"
- board text added: "J2"
- board text added: "J3"
- board text added: "J4"
- board text added: "JP2"
- board text added: "JP5"
- board text added: "PWR3"
- board text added: "Power"
- board text added: "Q1"
- board text added: "Q2"
- board text added: "Q3"
- board text added: "Q4"
- board text added: "Q5"
- board text added: "Q6"
- board text added: "Q7"
- board text added: "Q8"
- board text added: "R1"
- board text added: "R10"
- board text added: "R11"
- board text added: "R12"
- board text added: "R13"
- board text added: "R2"
- board text added: "R3"
- board text added: "R4"
- board text added: "R5"
- board text added: "R6"
- board text added: "R7"
- board text added: "R8"
- board text added: "R9"
- board text added: "RST"
- board text added: "RST0"
- board text added: "RST1"
- board text added: "SCL"
- board text added: "SDA"
- board text added: "SJ1"
- board text added: "SJ2"
- board text added: "SJ3"
- board text added: "SJ4"
- board text added: "SJ5"
- board text added: "TF"
- board text added: "TF0"
- board text added: "TF1"
- board text added: "TF2"
- board text added: "TF3"
- board text added: "U1"
- board text added: "VCC"
- board text added: "VccD"
- board text added: "VccH"
- board text added: "VccP"
- board text added: "X1"
- board text added: "XBP"
- board text added: "rev 2.0"
- board text removed: "XXBX Power Shim-XBP"
- board text removed: "rev 1.0"
