File: boards/xbp/XBP.brd (EAGLE design)
At the start: 61.3 x 31.1 mm, 41 parts, among them IC1 MCP1701AT, Q1 BSS84, Q2 BSS123, Q3 BSS123, Q4 BSS123, Q5 BSS123, Q6 BSS123, Q7 BSS123, Q8 BSS123, U1 INA225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

Commit message: added lots of stuff and updated class file too
Connections:
- net VCC renamed VCCH
Changed lines of the file:
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@@
 <wire x1="43.18" y1="2.9725" x2="43.18" y2="5.1825" width="0.254" layer="1"/>
 </signal>
-<signal name="VCC">
+<signal name="VCCH">
 <contactref element="Q1" pad="2"/>
 <contactref element="R4" pad="2"/>
