File: xbp/XBP.sch (EAGLE design)
At the start: 41 parts, among them IC1 MCP1701AT, Q1 BSS84, Q2 BSS123, Q3 BSS123, Q4 BSS123, Q5 BSS123, Q6 BSS123, Q7 BSS123, Q8 BSS123, U1 INA225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

Commit message: XBP version 2.1
Parts:
- removed U4: SILK_3V3_TAG, Public_BP_Library:SILK_3V3_TAG
Connections:
- net VCCXBD: now also JP2.4
Other:
- note added: "rev 2.1"
- note removed: "rev 2.0"
Changed lines of the file:
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@@
 <part name="U3" library="Public_BP_Library" deviceset="SILK_3V3_TAG" device=""/>
 <part name="A2" library="Public_BP_Library" deviceset="HEADER4X10-BOOSTERPACK" device="" value="XBDCon"/>
-<part name="U4" library="Public_BP_Library" deviceset="SILK_3V3_TAG" device=""/>
 <part name="U1" library="ina225" deviceset="INA225AIDGKR" device="" value="INA225"/>
 <part name="R1" library="resistor" deviceset="R-US_" device="R1210" value="1R"/>
@@
 <text x="149.86" y="30.48" size="3.81" layer="121">XXBX Power Shim - XBP</text>
 <text x="149.86" y="25.4" size="2.54" layer="121">cryptography.gmu.edu</text>
-<text x="236.22" y="7.62" size="2.54" layer="121">rev 2.0</text>
+<text x="236.22" y="7.62" size="2.54" layer="121">rev 2.1</text>
 </plain>
 <instances>
@@
 <instance part="U3" gate="G$1" x="109.22" y="170.18"/>
 <instance part="A2" gate="G$1" x="121.92" y="111.76"/>
-<instance part="U4" gate="G$1" x="109.22" y="124.46"/>
 <instance part="U1" gate="A" x="157.48" y="68.58"/>
 <instance part="R1" gate="G$1" x="121.92" y="73.66" rot="R180"/>
@@
 <wire x1="55.88" y1="73.66" x2="55.88" y2="55.88" width="0.1524" layer="91"/>
 <wire x1="12.7" y1="73.66" x2="55.88" y2="73.66" width="0.1524" layer="91"/>
-</segment>
-</net>
+<pinref part="JP2" gate="A" pin="4"/>
+<wire x1="20.32" y1="116.84" x2="48.26" y2="116.84" width="0.1524" layer="91"/>
+<wire x1="48.26" y1="116.84" x2="48.26" y2="109.22" width="0.1524" layer="91"/>
+<wire x1="48.26" y1="109.22" x2="58.42" y2="109.22" width="0.1524" layer="91"/>
+<wire x1="58.42" y1="109.22" x2="58.42" y2="78.74" width="0.1524" layer="91"/>
+<wire x1="58.42" y1="78.74" x2="55.88" y2="78.74" width="0.1524" layer="91"/>
+<wire x1="55.88" y1="78.74" x2="55.88" y2="73.66" width="0.1524" layer="91"/>
+<junction x="55.88" y="73.66"/>
+<label x="25.4" y="116.84" size="1.778" layer="95"/>
+</segment>
+</net>
